File: hw/zxkbd.sch (KiCad schematic (older format))
At the start: 56 parts, among them J1 TAPOUT, J2 TAPIN, J3 AY_IN, J4 SCART, J5 SERIAL, J6 ISP, Q1 BC846, SW1 RESET, SW2 MAGIC, SW3 AVR_RST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

Commit message: designing the pcb
Parts:
- removed J1: TAPOUT, Connector_PinHeader_2.54mm:PinHeader_1x02_P2.54mm_Horizontal, symbol Connector:AudioJack2
- removed J2: TAPIN, Connector_PinHeader_2.54mm:PinHeader_1x02_P2.54mm_Horizontal, symbol Connector:AudioJack2
- removed RN1, RN2, RN3, RN4, RN5, RN6: 4k7, Resistor_THT:R_Array_SIP9, symbol Device:R_Network08
- added J1: TAPE, Connector_PinHeader_2.54mm:PinHeader_1x03_P2.54mm_Vertical, symbol Connector_Generic:Conn_01x03
- added RN1, RN2, RN3, RN4, RN5, RN6: 4k7, Resistor_SMD:R_Array_Convex_5x1206, symbol zxkbd:R_Network08_SMD
- added unit 2 of U2
- added unit 2 of U3
- added unit 2 of U4
- added unit 2 of U5
- added unit 2 of U6
- U11: footprint (none) -> zxkbd:ps2conn
- U8: footprint Connector_PinHeader_2.54mm:PinHeader_2x32_P2.54mm_Vertical -> zxkbd:pentconn
Connections:
- wire segments 331 -> 341
- no-connect marks 28 -> 34

Commit message: finishing the pcb
Parts:
- added C15, C16, C17: 0.1uF, Capacitor_SMD:C_0805_2012Metric_Pad1.15x1.40mm_HandSolder, symbol Device:C_Small
Connections:
- wire segments 341 -> 347
Changed lines of the file:
@@
 Wire Wire Line
 	-2550 3250 -2050 3250
+Connection ~ -2050 3250
+Wire Wire Line
+	-2050 3250 -1550 3250
+Connection ~ -1550 3250
+Wire Wire Line
+	-1550 3250 -1050 3250
+Connection ~ -1050 3250
+Wire Wire Line
+	-1050 3250 -550 3250
+$Comp
+L Device:C_Small C15
+U 1 1 5F1D8CBC
+P 5050 7250
+F 0 "C15" H 5000 7450 50  0000 L CNN
+F 1 "0.1uF" H 4950 7050 50  0000 L CNN
+F 2 "Capacitor_SMD:C_0805_2012Metric_Pad1.15x1.40mm_HandSolder" H 5050 7250 50  0001 C CNN
+F 3 "~" H 5050 7250 50  0001 C CNN
+	1    5050 7250
+	1    0    0    -1
+$EndComp
+$Comp
+L Device:C_Small C16
+U 1 1 5F1D8CC6
+P 5300 7250
+F 0 "C16" H 5250 7450 50  0000 L CNN
+F 1 "0.1uF" H 5200 7050 50  0000 L CNN
+F 2 "Capacitor_SMD:C_0805_2012Metric_Pad1.15x1.40mm_HandSolder" H 5300 7250 50  0001 C CNN
+F 3 "~" H 5300 7250 50  0001 C CNN
+	1    5300 7250
+	1    0    0    -1
+$EndComp
+$Comp
+L Device:C_Small C17
+U 1 1 5F1D8CD0
+P 5550 7250
+F 0 "C17" H 5500 7450 50  0000 L CNN
+F 1 "0.1uF" H 5450 7050 50  0000 L CNN
+F 2 "Capacitor_SMD:C_0805_2012Metric_Pad1.15x1.40mm_HandSolder" H 5550 7250 50  0001 C CNN
+F 3 "~" H 5550 7250 50  0001 C CNN
+	1    5550 7250
+	1    0    0    -1
+$EndComp
+Wire Wire Line
+	4800 7150 5050 7150
+Connection ~ 4800 7150
+Connection ~ 5050 7150
+Wire Wire Line
+	5050 7150 5300 7150
+Connection ~ 5300 7150
+Wire Wire Line
+	5300 7150 5550 7150
+Wire Wire Line
+	4800 7350 5050 7350
+Connection ~ 4800 7350
+Connection ~ 5050 7350
+Wire Wire Line
+	5050 7350 5300 7350
+Connection ~ 5300 7350
+Wire Wire Line
+	5300 7350 5550 7350
 Wire Bus Line
 	7550 650  7550 1550
@@
 Wire Bus Line
 	9250 650  9250 6400
-Connection ~ -2050 3250
-Wire Wire Line
-	-2050 3250 -1550 3250
-Connection ~ -1550 3250
-Wire Wire Line
-	-1550 3250 -1050 3250
-Connection ~ -1050 3250
-Wire Wire Line
-	-1050 3250 -550 3250
 $EndSCHEMATC

Commit message: PCB completed
Parts:
- added J2: LINEOUT, zxkbd:cui_sj1-3525ng, symbol zxkbd:SJ1-3525NG
Connections:
- wire segments 347 -> 354
- no-connect marks 34 -> 37
Other:
- moved on the sheet: C1, C11, C15, C16, C17, C2, C3, C4, C5, C6, C7, C8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
